File: keeby cat.kicad_pcb (KiCad board)
At the start: 2 copper layers, 60 x 100 mm, 63 parts, among them SW1 SW_Push, SW10 SW_Push, SW11 SW_Push, SW12 SW_Push, SW13 SW_Push, SW14 SW_Push, SW15 SW_Push, SW2 SW_Push, SW3 SW_Push, SW4 SW_Push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

Commit message: routing improvements
Parts:
- added H5: MountingHole, Keeby-Cat Footprints:MountingHole_2.2mm_M2_DIN965, F.Cu at (101.7, 138.0)
- moved kibuzzard-6226FF10 3.69 mm to (113.2, 136.7)
Routing:
- net GND: track 66.0 -> 78.2 mm, vias 3 -> 4
- net KEY4: track 52.7 -> 41.1 mm
- net +3V3: track 102.0 -> 110.5 mm
- net Net-(D3-Pad2): track 42.7 -> 40.2 mm, vias 2 -> 3
- net SDA-SW: track 53.2 -> 55.3 mm
- net ENC3B: track 67.1 -> 65.0 mm
- net +5V: track 332.6 -> 330.5 mm, vias 19 -> 21
- net KEY7: track 60.1 -> 61.9 mm
- net Net-(D13-Pad2): track 28.1 -> 26.3 mm, vias 3 -> 0
- net Net-(D1-Pad2): track 50.1 -> 48.8 mm
- net Net-(D8-Pad2): track 81.9 -> 80.6 mm
- net KEY1: track 34.9 -> 36.2 mm
- net KEY12-POT2: track 70.1 -> 71.3 mm
- net Net-(D2-Pad2): track 47.5 -> 46.4 mm
- net KEY8: track 75.5 -> 76.5 mm
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Other:
- outline, holes or cut-outs redrawn
